Commit message: feat: configurable IMU position and yaw via mowgli_robot.yaml
Added imu_x, imu_y, imu_z, imu_yaw xacro args for the IMU joint,
same pattern as the lidar parameters. The IMU position affects
acceleration readings (centripetal acceleration during rotation)
and the yaw offset allows for IMUs mounted at an angle.

Defaults: centered at (0, 0, 0.095) with no rotation.

File: src/mowgli_bringup/urdf/mowgli.urdf.xacro (robot description, xacro)
@@ -24,4 +24,8 @@
   <xacro:arg name="lidar_z"   default="0.22"/>
   <xacro:arg name="lidar_yaw" default="0.0"/>
+  <xacro:arg name="imu_x"     default="0.0"/>
+  <xacro:arg name="imu_y"     default="0.0"/>
+  <xacro:arg name="imu_z"     default="0.095"/>
+  <xacro:arg name="imu_yaw"   default="0.0"/>
   <!-- ================================================================
        Properties
@@ -268,5 +272,5 @@
     <parent link="base_link"/>
     <child  link="imu_link"/>
-    <origin xyz="0 0 ${base_height/2}" rpy="0 0 0"/>
+    <origin xyz="$(arg imu_x) $(arg imu_y) $(arg imu_z)" rpy="0 0 $(arg imu_yaw)"/>
   </joint>
   <!-- ================================================================

Commit message: feat: configurable GPS antenna position via mowgli_robot.yaml

File: src/mowgli_bringup/urdf/mowgli.urdf.xacro (robot description, xacro)
@@ -28,4 +28,7 @@
   <xacro:arg name="imu_z"     default="0.095"/>
   <xacro:arg name="imu_yaw"   default="0.0"/>
+  <xacro:arg name="gps_x"     default="0.0"/>
+  <xacro:arg name="gps_y"     default="0.0"/>
+  <xacro:arg name="gps_z"     default="0.20"/>
   <!-- ================================================================
        Properties
@@ -303,6 +306,5 @@
     <parent link="base_link"/>
     <child  link="gps_link"/>
-    <!-- Mounted on top surface, centred -->
-    <origin xyz="0 0 ${base_height + 0.01}" rpy="0 0 0"/>
+    <origin xyz="$(arg gps_x) $(arg gps_y) $(arg gps_z)" rpy="0 0 0"/>
   </joint>
   <!-- ================================================================
